Commit message: added color to the models, updeated the control launch file

File: urdf/r2d2.xacro (robot description, xacro)
@@ -37,4 +37,7 @@
     <xacro:default_inertial mass="10"/>
   </link>
+  <gazebo reference="base_link">
+    <material>Gazebo/Blue</material>
+  </gazebo>
   <xacro:macro name="wheel" params="prefix suffix reflect">
     <link name="${prefix}_${suffix}_wheel">
@@ -100,4 +103,7 @@
       <xacro:default_inertial mass="10"/>
     </link>
+    <gazebo reference="${prefix}_leg">
+      <material>Gazebo/White</material>
+    </gazebo>
     <joint name="base_to_${prefix}_leg" type="fixed">
       <parent link="base_link"/>
@@ -119,4 +125,7 @@
       <xacro:default_inertial mass="10"/>
     </link>
+    <gazebo reference="${prefix}_base">
+      <material>Gazebo/White</material>
+    </gazebo>
     <joint name="${prefix}_base_joint" type="fixed">
       <parent link="${prefix}_leg"/>
@@ -231,4 +240,7 @@
     <xacro:default_inertial mass="2"/>
   </link>
+  <gazebo reference="head">
+    <material>Gazebo/White</material>
+  </gazebo>
   <joint name="head_swivel" type="continuous">
     <parent link="base_link"/>
@@ -265,4 +277,7 @@
     <xacro:default_inertial mass="1"/>
   </link>
+  <gazebo reference="box">
+    <material>Gazebo/Blue</material>
+  </gazebo>
   <joint name="tobox" type="fixed">
     <parent link="head"/>
