Commit message: Correctly sized wheels that work in gazebo, simulation works in gazebo

File: urdf/traditionalApproach2016.urdf (robot description, URDF)
Before this commit: robot traditional_2016, 10 links, 9 joints
Links:
- added link left_front_wheel, mass 1.05364116667; collision cylinder length=0.118 radius=0.15; visual cylinder length=0.118 radius=0.15
- added link left_rear_wheel, mass 1.05364116667; collision cylinder length=0.118 radius=0.15; visual cylinder length=0.118 radius=0.15
- added link offsetMass, mass 3; collision box size=0 0 0; visual box size=0 0 0
- added link right_front_wheel, mass 1.05364116667; collision cylinder length=0.118 radius=0.15; visual cylinder length=0.118 radius=0.15
- added link right_rear_wheel, mass 1.05364116667; collision cylinder length=0.118 radius=0.15; visual cylinder length=0.118 radius=0.15
- link Front Piece: mass 0.239915601207774 -> 0.01
- link Sideplate Frame: mass 4.69519028792857 -> 0.1
- link base_link: mass 4.21456466669016 -> 1; geometry collision box size=0.1 0.1 0.1; visual box size=0.1 0.1 0.1
Joints:
- removed joint Front Piece Joint
- removed joint Sideplate Frame Joint
- added joint Front_Piece_Joint: type revolute, parent Sideplate Frame, child Front Piece, origin xyz=1.1653 0.044207 0 rpy=0.78967 -1.5708 0, axis -1 0 0, limit lower=-2.935619449019 upper=-1.57079632679 effort=0 velocity=0
- added joint Sideplate_Frame_Joint: type revolute, parent Chassis, child Sideplate Frame, origin xyz=-0.21821 0.39829 0 rpy=0 0 0.44824, axis 0 0 -1, limit lower=-.25 upper=1 effort=0 velocity=0
- added joint left_front_wheel_joint: type continuous, parent base_link, child left_front_wheel, origin xyz=0.47 0.247 -0.078 rpy=0 0 0, axis 0 1 0
- added joint left_rear_wheel_joint: type continuous, parent base_link, child left_rear_wheel, origin xyz=-0.06 0.247 -0.078 rpy=0 0 0, axis 0 1 0
- added joint offsetMass_joint: type fixed, parent Chassis, child offsetMass, origin xyz=0.54 0 0
- added joint right_front_wheel_joint: type continuous, parent base_link, child right_front_wheel, origin xyz=0.47 -0.38 -0.078 rpy=0 0 0, axis 0 1 0
- added joint right_rear_wheel_joint: type continuous, parent base_link, child right_rear_wheel, origin xyz=-0.06 -0.38 -0.078 rpy=0 0 0, axis 0 1 0
- joint tokinect: origin xyz=0.52 0.35 -0.25 rpy=0 3.1415926535897931 3.1415926535897931 -> xyz=0.52 0.35 -0.25 rpy=0 3.1415926535897931 2.8

Commit message: Added meshes for kinect

File: urdf/traditionalApproach2016.urdf (robot description, URDF)
Before this commit: robot traditional_2016, 15 links, 14 joints
Links:
- link camera_link: geometry collision box size=0.07271 0.27794 0.073; visual mesh filename=package://gazebo_sim/meshes/kinect.dae
